File: my-prj/16X2LCD_SIMPLE_SPI/16X2LCD_SIMPLE_SPI.sch (EAGLE design)
At the start: 10 parts, among them IC1 4094D, U1 LCD-16X2SILK

Commit message: t
Parts:
- removed JP3, JP4: (no value), SparkFun-Connectors:M041.27MM
- removed JP5, JP6: (no value), SparkFun:M04LOCK_LONGPADS
- removed R3: TRIMPOT, SparkFun:TRIMPOT
- added U$1: TRIMPOT_S3_SMD, custom:TRIMPOT_S3_SMD
- D1: device SparkFun:DIODE1N4148 -> SparkFun-DiscreteSemi:DIODESMA
- R1: device SparkFun:RESISTORAXIAL-0.3 -> SparkFun-Passives:RESISTOR1206
Connections:
- removed net N$11: JP3.3, JP5.2
- removed net N$12: JP3.4, JP5.1
- removed net N$13: JP4.1, JP6.4
- removed net N$14: JP4.2, JP6.3
- removed net N$15: JP4.3, JP6.2
- removed net N$16: JP4.4, JP6.1
- removed net N$5: JP3.1, JP5.4
- removed net N$8: JP3.2, JP5.3
- net CLK: now also JP1.2; no longer JP1.3
- net DATA: now also JP1.3; no longer JP1.4
- net GND: now also U$1.CCW; no longer R3.CCW
- net N$3: now also U$1.WIPER; no longer R3.WIPER
- net VDD: now also JP1.4, U$1.CW; no longer JP1.2, R3.CW
Other:
- moved on the sheet: JP1
Changed lines of the file:
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@@
 <?xml version="1.0" encoding="utf-8"?>
 <!DOCTYPE eagle SYSTEM "eagle.dtd">
-<eagle version="6.3">
+<eagle version="6.4">
 <drawing>
 <settings>
@@
 <layer number="106" name="bPlate" color="7" fill="1" visible="no" active="yes"/>
 <layer number="107" name="Crop" color="7" fill="1" visible="no" active="yes"/>
+<layer number="108" name="fp8" color="7" fill="1" visible="yes" active="yes"/>
+<layer number="109" name="fp9" color="7" fill="1" visible="yes" active="yes"/>
+<layer number="110" name="fp0" color="7" fill="1" visible="yes" active="yes"/>
 <layer number="116" name="Patch_BOT" color="9" fill="4" visible="no" active="yes"/>
 <layer number="121" name="_tsilk" color="7" fill="1" visible="no" active="yes"/>
 <layer number="122" name="_bsilk" color="7" fill="1" visible="no" active="yes"/>
+<layer number="123" name="tTestmark" color="7" fill="1" visible="yes" active="yes"/>
+<layer number="124" name="bTestmark" color="7" fill="1" visible="yes" active="yes"/>
 <layer number="125" name="_tNames" color="7" fill="1" visible="no" active="yes"/>
+<layer number="131" name="tAdjust" color="7" fill="1" visible="yes" active="yes"/>
+<layer number="132" name="bAdjust" color="7" fill="1" visible="yes" active="yes"/>
 <layer number="144" name="Drill_legend" color="7" fill="1" visible="no" active="yes"/>
 <layer number="151" name="HeatSink" color="7" fill="1" visible="no" active="yes"/>
@@
 <part name="GND3" library="SparkFun" deviceset="GND" device=""/>
 <part name="P+1" library="SparkFun" deviceset="VCC" device=""/>
-<part name="R1" library="SparkFun" deviceset="RESISTOR" device="AXIAL-0.3"/>
-<part name="D1" library="SparkFun" deviceset="DIODE" device="1N4148"/>
+<part name="R1" library="SparkFun-Passives" deviceset="RESISTOR" device="1206"/>
+<part name="D1" library="SparkFun-DiscreteSemi" deviceset="DIODE" device="SMA"/>
 <part name="JP1" library="SparkFun" deviceset="M04" device="PTH"/>
 <part name="VDD1" library="supply1" deviceset="VDD" device=""/>
 <part name="VSS1" library="supply1" deviceset="VSS" device=""/>
 <part name="GND2" library="SparkFun" deviceset="GND" device=""/>
-<part name="R3" library="SparkFun" deviceset="TRIMPOT" device=""/>
-<part name="JP3" library="SparkFun-Connectors" deviceset="M04" device="1.27MM"/>
-<part name="JP4" library="SparkFun-Connectors" deviceset="M04" device="1.27MM"/>
-<part name="JP5" library="SparkFun" deviceset="M04" device="LOCK_LONGPADS"/>
-<part name="JP6" library="SparkFun" deviceset="M04" device="LOCK_LONGPADS"/>
+<part name="U$1" library="custom" deviceset="TRIMPOT_S3_SMD" device=""/>
 </parts>
 <sheets>
@@
 <instance part="R1" gate="G$1" x="71.12" y="-53.34"/>
 <instance part="D1" gate="G$1" x="71.12" y="-33.02" rot="R180"/>
-<instance part="JP1" gate="G$1" x="-35.56" y="-45.72"/>
+<instance part="JP1" gate="G$1" x="-30.48" y="-43.18" rot="MR180"/>
 <instance part="VDD1" gate="G$1" x="-27.94" y="27.94"/>
 <instance part="VSS1" gate="G$1" x="-27.94" y="45.72"/>
-<instance part="GND2" gate="1" x="-17.78" y="-55.88"/>
-<instance part="R3" gate="R?" x="132.08" y="7.62" rot="R90"/>
-<instance part="JP3" gate="G$1" x="187.96" y="-15.24" rot="R180"/>
-<instance part="JP4" gate="G$1" x="187.96" y="-38.1" rot="R180"/>
-<instance part="JP5" gate="G$1" x="147.32" y="-17.78"/>
-<instance part="JP6" gate="G$1" x="147.32" y="-40.64"/>
+<instance part="GND2" gate="1" x="-17.78" y="-30.48" rot="R180"/>
+<instance part="U$1" gate="G$1" x="132.08" y="7.62" rot="R90"/>
 </instances>
 <busses>
@@
 <segment>
 <pinref part="GND1" gate="1" pin="GND"/>
-<wire x1="132.08" y1="5.08" x2="132.08" y2="2.54" width="0.1524" layer="91"/>
-<pinref part="R3" gate="R?" pin="CCW"/>
 <wire x1="132.08" y1="2.54" x2="132.08" y2="-7.62" width="0.1524" layer="91"/>
-<junction x="132.08" y="2.54"/>
-</segment>
-<segment>
-<pinref part="JP1" gate="G$1" pin="1"/>
-<pinref part="GND2" gate="1" pin="GND"/>
-<wire x1="-30.48" y1="-48.26" x2="-17.78" y2="-48.26" width="0.1524" layer="91"/>
-<wire x1="-17.78" y1="-48.26" x2="-17.78" y2="-53.34" width="0.1524" layer="91"/>
+<pinref part="U$1" gate="G$1" pin="CCW"/>
 </segment>
 <segment>
@@
 <junction x="106.68" y="40.64"/>
 </segment>
+<segment>
+<pinref part="JP1" gate="G$1" pin="1"/>
+<pinref part="GND2" gate="1" pin="GND"/>
+<wire x1="-25.4" y1="-40.64" x2="-17.78" y2="-40.64" width="0.1524" layer="91"/>
+<wire x1="-17.78" y1="-40.64" x2="-17.78" y2="-33.02" width="0.1524" layer="91"/>
+</segment>
 </net>
 <net name="N$3" class="0">
@@
 <pinref part="U1" gate="G$1" pin="VO"/>
 <wire x1="88.9" y1="7.62" x2="88.9" y2="45.72" width="0.1524" layer="91"/>
-<pinref part="R3" gate="R?" pin="WIPER"/>
 <wire x1="88.9" y1="7.62" x2="127" y2="7.62" width="0.1524" layer="91"/>
+<pinref part="U$1" gate="G$1" pin="WIPER"/>
 </segment>
 </net>
@@
 <net name="DATA" class="0">
 <segment>
+<pinref part="JP1" gate="G$1" pin="3"/>
 <pinref part="R1" gate="G$1" pin="1"/>
 <wire x1="66.04" y1="-53.34" x2="2.54" y2="-53.34" width="0.1524" layer="91"/>
@@
 <pinref part="IC1" gate="A" pin="D"/>
 <wire x1="7.62" y1="-45.72" x2="2.54" y2="-45.72" width="0.1524" layer="91"/>
-</segment>
-<segment>
-<wire x1="-17.78" y1="-40.64" x2="-30.48" y2="-40.64" width="0.1524" layer="91"/>
-<pinref part="JP1" gate="G$1" pin="4"/>
+<wire x1="-25.4" y1="-45.72" x2="2.54" y2="-45.72" width="0.1524" layer="91"/>
+<junction x="2.54" y="-45.72"/>
 </segment>
 </net>
@@
 <segment>
 <pinref part="IC1" gate="A" pin="CLK"/>
-<wire x1="7.62" y1="-43.18" x2="2.54" y2="-43.18" width="0.1524" layer="91"/>
-</segment>
-<segment>
-<pinref part="JP1" gate="G$1" pin="3"/>
-<wire x1="-30.48" y1="-43.18" x2="-17.78" y2="-43.18" width="0.1524" layer="91"/>
+<pinref part="JP1" gate="G$1" pin="2"/>
+<wire x1="-25.4" y1="-43.18" x2="7.62" y2="-43.18" width="0.1524" layer="91"/>
 </segment>
 </net>
@@
 <wire x1="-27.94" y1="22.86" x2="-2.54" y2="22.86" width="0.1524" layer="91"/>
 <junction x="-2.54" y="22.86"/>
-<pinref part="R3" gate="R?" pin="CW"/>
 <wire x1="119.38" y1="22.86" x2="132.08" y2="22.86" width="0.1524" layer="91"/>
 <wire x1="132.08" y1="22.86" x2="132.08" y2="12.7" width="0.1524" layer="91"/>
 <junction x="119.38" y="22.86"/>
-</segment>
-<segment>
-<pinref part="JP1" gate="G$1" pin="2"/>
-<wire x1="-30.48" y1="-45.72" x2="-17.78" y2="-45.72" width="0.1524" layer="91"/>
-</segment>
-</net>
-<net name="N$5" class="0">
-<segment>
-<pinref part="JP5" gate="G$1" pin="4"/>
-<pinref part="JP3" gate="G$1" pin="1"/>
-<wire x1="152.4" y1="-12.7" x2="182.88" y2="-12.7" width="0.1524" layer="91"/>
-</segment>
-</net>
-<net name="N$8" class="0">
-<segment>
-<pinref part="JP5" gate="G$1" pin="3"/>
-<pinref part="JP3" gate="G$1" pin="2"/>
-<wire x1="152.4" y1="-15.24" x2="182.88" y2="-15.24" width="0.1524" layer="91"/>
-</segment>
-</net>
-<net name="N$11" class="0">
-<segment>
-<pinref part="JP5" gate="G$1" pin="2"/>
-<pinref part="JP3" gate="G$1" pin="3"/>
-<wire x1="152.4" y1="-17.78" x2="182.88" y2="-17.78" width="0.1524" layer="91"/>
-</segment>
-</net>
-<net name="N$12" class="0">
-<segment>
-<pinref part="JP5" gate="G$1" pin="1"/>
-<pinref part="JP3" gate="G$1" pin="4"/>
-<wire x1="152.4" y1="-20.32" x2="182.88" y2="-20.32" width="0.1524" layer="91"/>
-</segment>
-</net>
-<net name="N$13" class="0">
-<segment>
-<pinref part="JP6" gate="G$1" pin="4"/>
-<pinref part="JP4" gate="G$1" pin="1"/>
-<wire x1="152.4" y1="-35.56" x2="182.88" y2="-35.56" width="0.1524" layer="91"/>
-</segment>
-</net>
-<net name="N$14" class="0">
-<segment>
-<pinref part="JP6" gate="G$1" pin="3"/>
-<pinref part="JP4" gate="G$1" pin="2"/>
-<wire x1="152.4" y1="-38.1" x2="182.88" y2="-38.1" width="0.1524" layer="91"/>
-</segment>
-</net>
-<net name="N$15" class="0">
-<segment>
-<pinref part="JP6" gate="G$1" pin="2"/>
-<pinref part="JP4" gate="G$1" pin="3"/>
-<wire x1="152.4" y1="-40.64" x2="182.88" y2="-40.64" width="0.1524" layer="91"/>
-</segment>
-</net>
-<net name="N$16" class="0">
-<segment>
-<pinref part="JP6" gate="G$1" pin="1"/>
-<pinref part="JP4" gate="G$1" pin="4"/>
-<wire x1="152.4" y1="-43.18" x2="182.88" y2="-43.18" width="0.1524" layer="91"/>
-</segment>
-</net>
+<pinref part="U$1" gate="G$1" pin="CW"/>
+<pinref part="JP1" gate="G$1" pin="4"/>
+<wire x1="-25.4" y1="-48.26" x2="-2.54" y2="-48.26" width="0.1524" layer="91"/>
+<junction x="-2.54" y="-48.26"/>
+</segment>
+</net>
