File: my-prj/MSP430_NRF24L01/BATCH_V1_1.brd (EAGLE design)
At the start: 49.5 x 25.4 mm, 20 parts, among them U1 NRF24L01-4X2

Commit message: adding new files
Parts:
- removed LED-P3.1: (no value), custom:LED-0805
- removed R103, R104: 47K, SparkFun-Resistors:0805
- added C3, C4: 0.1uF, SparkFun-Capacitors:0805
- added C5: 10uF, SparkFun-Capacitors:0805
- added JP4, JP5, JP7: (no value), SparkFun-Connectors:1X04_LOCK
- added JP6: (no value), SparkFun-Connectors:1X05_LOCK
- added L2, R5, R6: (no value), SparkFun-Passives:0805
- added LED-P1.0, LED-P1.1, RXLED, TXLED: (no value), custom:LED-0805
- added R11, R7: 220, SparkFun-Resistors:0805
- added R12, R13: 330, SparkFun-Passives:0805
- added U$3: G2XX3---PW28, TI_MSP430_v16:PW28
- added U2: NRF24L01-4X2, untitled:NRF24L01-4X2
- added U3: FT232RL-BASICSSOP, SparkFun-DigitalIC:SSOP28DB
- JP1: value (none) -> M05X2PTH; device SparkFun-Connectors:1X06_LOCK -> SparkFun-Connectors:AVR_ICSP
- JP2: value M05X2PTH -> (none); device SparkFun-Connectors:AVR_ICSP -> SparkFun-Connectors:1X06_LOCK
- JP3: value (none) -> USB-B; device SparkFun-Connectors:1X04_LOCK -> SparkFun-Connectors:USB-A-H
- R1, R2: value (none) -> 47K; device SparkFun-Passives:0805 -> SparkFun-Resistors:0805
- R3: value 220 -> 47K
- U$1: value TLV61220 -> G2XX3---PW28; device custom:SOT23-6L -> TI_MSP430_v16:PW28
- U$2: value MSP430G2553 -> TI-TLV61220; device TI_MSP430_v16:PW28 -> custom:SOT23-6L
- moved U$1 40.0 mm to (34.9, 39.4), turned to 0 degrees
- moved R1 31.9 mm to (34.3, 29.8), turned to 90 degrees
- moved U$2 30.7 mm to (5.08, 12.7), turned to 90 degrees
- moved JP3 28.8 mm to (3.81, 36.8), turned to 0 degrees
- moved U1 27.9 mm to (33.7, 39.4), turned to 180 degrees
- moved R2 17.8 mm to (24.8, 18.4)
- moved R4 13.3 mm to (39.4, 15.9), flipped to the bottom, turned to 90 degrees
- moved R3 13.0 mm to (36.8, 15.9), flipped to the bottom, turned to 90 degrees
- moved C1 8.89 mm to (3.17, 8.26), turned to 270 degrees
- moved C2 8.89 mm to (3.17, 17.1), turned to 90 degrees
- moved JP2 8.35 mm to (33.7, 23.5), turned to 180 degrees
- moved JP1 8.25 mm to (41.9, 22.2), turned to 270 degrees
- renumbered R100 to R9, R101 to R10, R102 to R8
Connections:
- new net 5V: C5.1, JP6.5, L2.2, R12.1, R13.1, U3.20
- new net GND1: C3.2, C4.2, C5.2, JP3.VBUS, JP4.1, JP6.1, JP7.1, LED-P1.1.C, U$1.28, U1.1, U3.18, U3.21, U3.25, U3.26, U3.7
- new net N$10: R12.2, TXLED.A
- new net N$11: TXLED.C, U3.23
- new net N$12: U$1.10, U1.8
- new net N$16: C4.1, JP3.GND, L2.1
- new net N$2: U$1.18, U1.3
- new net N$24: R11.1, U$1.2
- new net N$3: U$1.17, U1.5
- new net N$4: U$1.16, U1.7
- new net N$5: U$1.11, U1.6
- new net N$6: U$1.12, U1.4
- new net N$7: R13.2, RXLED.A
- new net N$8: LED-P1.1.A, R11.2
- new net N$9: RXLED.C, U3.22
- new net RESET1: JP4.3, R1.1, U$1.24
- new net RX: JP6.3, JP7.3, U$1.4, U3.5
- new net TEST1: JP4.2, U$1.25
- new net TX: JP6.2, JP7.2, U$1.3, U3.1
- new net USBDM: JP3.D-, U3.16
- new net USBDP: JP3.D+, U3.15
- new net VCC1: C3.1, JP4.4, JP6.4, JP7.4, R1.2, U$1.1, U1.2, U3.17, U3.4
- net GND: now also JP1.1, JP1.3, JP1.5, JP1.7, JP1.9, JP2.6, JP5.1, LED-P1.0.C, R5.1, U$2.2, U$3.28, U2.1; no longer JP1.6, JP2.1, JP2.3, JP2.5, JP2.7, JP2.9, JP3.1, LED-P3.1.C, R2.1, U$1.2, U$2.28, U1.1
- net N$1: now also R3.1, R4.1, U$3.8; no longer R103.1, R104.1, U$2.8
- net N$13: now also U$2.1; no longer U$1.1
- net N$14: now also R5.2, R6.1, U$2.4; no longer R1.1, R2.2, U$1.4
- net N$15: now also LED-P1.0.A, R7.2; no longer LED-P3.1.A, R3.2
- net N$17: now also U$3.18, U2.3; no longer U$2.18, U1.3
- net N$18: now also U$3.17, U2.5; no longer U$2.17, U1.5
- net N$19: now also U$3.16, U2.7; no longer U$2.16, U1.7
- net N$20: now also U$3.11, U2.6; no longer U$2.11, U1.6
- net N$21: now also U$3.12, U2.4; no longer U$2.12, U1.4
- net N$22: now also U$3.10, U2.8; no longer U$2.10, U1.8
- net N$23: now also R7.1, U$3.9; no longer R3.1, U$2.9
- net P1.0: now also JP1.8, R4.2, U$3.2; no longer JP2.8, R103.2, U$2.2
- net P1.3: now also JP1.6, U$3.5; no longer JP2.6, U$2.5
- net P1.4: now also JP1.4, U$3.6; no longer JP2.4, U$2.6
- net P1.5: now also JP1.2, U$3.7; no longer JP2.2, U$2.7
- net P1.6: now also JP1.10, R3.2, U$3.22; no longer JP2.10, R104.2, U$2.22
- net RESET: now also JP2.5, R2.1, U$3.24; no longer JP1.5, R4.1, U$2.24
- net RXD: now also JP2.2, U$3.3; no longer JP1.2, U$2.3
- net TEST: now also JP2.4, U$3.25; no longer JP1.4, U$2.25
- net TXD: now also JP2.3, U$3.4; no longer JP1.3, U$2.4
- net VCC: now also C2.1, JP2.1, JP5.4, R2.2, R6.2, U$2.5, U$3.1, U2.2; no longer C1.1, JP1.1, JP3.4, R1.2, R4.2, U$1.5, U$2.1, U1.2
- net VIN: now also C1.1, JP5.2, U$2.3, U$2.6; no longer C2.1, JP3.2, U$1.3, U$1.6
Routing:
- net VCC1: track 0.00 -> 66.5 mm, vias 0 -> 3
- net 5V: track 0.00 -> 39.1 mm, vias 0 -> 3
- net RX: track 0.00 -> 36.7 mm, vias 0 -> 2
- net RESET1: track 0.00 -> 26.9 mm, vias 0 -> 2
- net TX: track 0.00 -> 26.4 mm, vias 0 -> 1
- net N$2: track 0.00 -> 25.9 mm, vias 0 -> 1
- net TEST1: track 0.00 -> 24.1 mm, vias 0 -> 1
- net GND1: track 0.00 -> 21.6 mm
- net N$3: track 0.00 -> 17.5 mm
- net N$12: track 0.00 -> 10.6 mm
- net N$4: track 0.00 -> 10.2 mm
- net USBDP: track 0.00 -> 8.88 mm, vias 0 -> 2
- net N$5: track 0.00 -> 8.49 mm
- net N$10: track 0.00 -> 6.76 mm
- net USBDM: track 0.00 -> 6.76 mm
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- added copper zone on layer 1, net GND1
- added copper zone on layer 16, net GND1
Other:
- board size 49.5 x 25.4 mm -> 49.2 x 48.2 mm
- board text added: "3V3"
- board text added: "5V"
- board text added: "FTDI USB <=> UART TTL V1"
- board text added: "MSP430 RF V1"
- board text added: "RST"
- board text added: "RX"
- board text added: "TST"
- board text added: "TX"
- board text removed: "RESET"
- board text removed: "TEST"
