File: my-prj/MSP430_NRF24L01/V1_HUB.brd (EAGLE design)
At the start: 49.8 x 22.9 mm, 18 parts, among them U1 NRF24L01-4X2, U2 FT232RL-BASICSSOP

Commit message: adding new files
Parts:
- removed JP5: (no value), SparkFun-Connectors:1X04_LOCK
- added JP1: USB-B, SparkFun-Connectors:USB-A-H
- JP3: value USB-B -> (none); device SparkFun-Connectors:USB-A-H -> SparkFun-Connectors:1X04_LOCK
- R2: value 47K -> 330; device SparkFun-Resistors:0805 -> SparkFun-Passives:0805
- R3: value 330 -> 220; device SparkFun-Passives:0805 -> SparkFun-Resistors:0805
- R4: value 220 -> 47K
- moved JP3 24.7 mm to (27.9, 6.35), turned to 90 degrees
- moved R2 21.6 mm to (12.7, 4.45)
- moved R3 19.7 mm to (32.4, 4.45)
- moved C1 10.2 mm to (8.26, 18.4)
- moved C3 10.2 mm to (18.4, 18.4)
- moved R1 7.62 mm to (18.4, 4.45), turned to 90 degrees
- moved R4 1.91 mm to (34.3, 4.45), turned to 90 degrees
- renumbered LED-P1.0 to LED-P1.1
Connections:
- net 5V: now also R2.1; no longer R3.1
- net GND: now also JP1.GND, JP3.1; no longer JP3.VBUS, JP5.1
- net N$13: now also R2.2; no longer R3.2
- net N$16: now also C1.1, JP1.VBUS; no longer C3.1, JP3.GND
- net N$4: now also R3.1; no longer R4.1
- net N$8: now also R3.2; no longer R4.2
- net RESET: now also R4.1; no longer R2.1
- net RX: now also JP3.3; no longer JP5.3
- net TX: now also JP3.2; no longer JP5.2
- net USBDM: now also JP1.D-; no longer JP3.D-
- net USBDP: now also JP1.D+; no longer JP3.D+
- net VCC: now also C3.1, JP3.4, R4.2; no longer C1.1, JP5.4, R2.2
Routing:
- net N$16: track 5.98 -> 15.5 mm, vias 0 -> 1
- net USBDP: track 8.88 -> 14.6 mm
- net N$10: track 6.76 -> 2.62 mm
- net VCC: track 65.6 -> 62.0 mm
- net 5V: track 39.1 -> 41.8 mm
- net N$13: track 1.91 -> 2.62 mm
- net GND: vias 0 -> 1
