File: my-prj/MSP430_NRF24L01/V1_HUB.sch (EAGLE design)
At the start: 18 parts, among them U1 NRF24L01-4X2, U2 FT232RL-BASICSSOP

Commit message: adding new files
Parts:
- removed JP5: (no value), SparkFun-Connectors:M04LOCK
- added JP1: USB-B, SparkFun-Connectors:USB-A-H
- JP3: value USB-B -> (none); device SparkFun-Connectors:USB-A-H -> SparkFun-Connectors:M04LOCK
- R2: value 47K -> 330; device SparkFun-Resistors:RESISTOR0805-RES -> SparkFun-Passives:RESISTOR0805-RES
- R3: value 330 -> 220; device SparkFun-Passives:RESISTOR0805-RES -> SparkFun-Resistors:RESISTOR0805-RES
- R4: value 220 -> 47K
- renumbered LED-P1.0 to LED-P1.1
Connections:
- net 5V: now also R2.1; no longer R3.1
- net GND: now also JP1.VBUS, JP3.1; no longer JP3.GND, JP5.1
- net N$13: now also R2.2; no longer R3.2
- net N$16: now also C1.1, JP1.GND; no longer C3.1, JP3.VBUS
- net N$4: now also R3.1; no longer R4.1
- net N$8: now also R3.2; no longer R4.2
- net RESET: now also R4.1; no longer R2.1
- net RX: now also JP3.3; no longer JP5.3
- net TX: now also JP3.2; no longer JP5.2
- net USBDM: now also JP1.D+; no longer JP3.D+
- net USBDP: now also JP1.D-; no longer JP3.D-
- net VCC: now also C3.1, JP3.4, R4.2; no longer C1.1, JP5.4, R2.2
Other:
- moved on the sheet: C1, C3, R2, R3, R4
Changed lines of the file:
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@@
 <part name="GND1" library="SparkFun-Aesthetics" deviceset="GND" device=""/>
 <part name="SUPPLY3" library="SparkFun-Aesthetics" deviceset="VCC" device=""/>
-<part name="R2" library="SparkFun-Resistors" deviceset="RESISTOR" device="0805-RES" value="47K"/>
+<part name="R4" library="SparkFun-Resistors" deviceset="RESISTOR" device="0805-RES" value="47K"/>
 <part name="SUPPLY4" library="SparkFun-Aesthetics" deviceset="VCC" device=""/>
 <part name="GND5" library="SparkFun-Aesthetics" deviceset="GND" device=""/>
-<part name="LED-P1.0" library="custom" deviceset="LED" device="0805"/>
-<part name="R4" library="SparkFun-Resistors" deviceset="RESISTOR" device="0805-RES" value="220"/>
+<part name="LED-P1.1" library="custom" deviceset="LED" device="0805"/>
+<part name="R3" library="SparkFun-Resistors" deviceset="RESISTOR" device="0805-RES" value="220"/>
 <part name="U2" library="SparkFun-DigitalIC" deviceset="FT232RL-BASIC" device="SSOP"/>
+<part name="C3" library="SparkFun-Capacitors" deviceset="CAP" device="0805" value="0.1uF"/>
 <part name="C1" library="SparkFun-Capacitors" deviceset="CAP" device="0805" value="0.1uF"/>
-<part name="C3" library="SparkFun-Capacitors" deviceset="CAP" device="0805" value="0.1uF"/>
-<part name="JP3" library="SparkFun-Connectors" deviceset="USB" device="-A-H" value="USB-B"/>
+<part name="JP1" library="SparkFun-Connectors" deviceset="USB" device="-A-H" value="USB-B"/>
 <part name="JP4" library="SparkFun-Connectors" deviceset="M04" device="LOCK"/>
 <part name="GND3" library="SparkFun-Aesthetics" deviceset="GND" device=""/>
@@
 <part name="GND6" library="SparkFun-Aesthetics" deviceset="GND" device=""/>
 <part name="R1" library="SparkFun-Passives" deviceset="RESISTOR" device="0805-RES" value="330"/>
-<part name="R3" library="SparkFun-Passives" deviceset="RESISTOR" device="0805-RES" value="330"/>
+<part name="R2" library="SparkFun-Passives" deviceset="RESISTOR" device="0805-RES" value="330"/>
 <part name="TXLED" library="custom" deviceset="LED" device="0805"/>
 <part name="RXLED" library="custom" deviceset="LED" device="0805"/>
@@
 <part name="C2" library="SparkFun-Capacitors" deviceset="CAP" device="0805" value="10uF"/>
 <part name="JP2" library="SparkFun-Connectors" deviceset="M05" device="LOCK"/>
-<part name="JP5" library="SparkFun-Connectors" deviceset="M04" device="LOCK"/>
+<part name="JP3" library="SparkFun-Connectors" deviceset="M04" device="LOCK"/>
 </parts>
 <sheets>
@@
 <instance part="GND1" gate="1" x="212.09" y="8.89"/>
 <instance part="SUPPLY3" gate="1" x="166.37" y="11.43" rot="R180"/>
-<instance part="R2" gate="G$1" x="224.79" y="77.47" rot="MR90"/>
+<instance part="R4" gate="G$1" x="224.79" y="77.47" rot="MR90"/>
 <instance part="SUPPLY4" gate="1" x="224.79" y="88.9" rot="MR0"/>
 <instance part="GND5" gate="1" x="115.57" y="41.91" rot="MR0"/>
-<instance part="LED-P1.0" gate="G$1" x="115.57" y="60.96" rot="MR0"/>
-<instance part="R4" gate="G$1" x="115.57" y="73.66" rot="MR270"/>
+<instance part="LED-P1.1" gate="G$1" x="115.57" y="60.96" rot="MR0"/>
+<instance part="R3" gate="G$1" x="115.57" y="73.66" rot="MR270"/>
 <instance part="U2" gate="G$1" x="40.64" y="40.64"/>
-<instance part="C1" gate="G$1" x="0" y="27.94"/>
-<instance part="C3" gate="G$1" x="22.86" y="91.44"/>
-<instance part="JP3" gate="G$1" x="2.54" y="106.68" rot="R180"/>
+<instance part="C3" gate="G$1" x="0" y="27.94"/>
+<instance part="C1" gate="G$1" x="22.86" y="91.44"/>
+<instance part="JP1" gate="G$1" x="0" y="104.14" rot="R180"/>
 <instance part="JP4" gate="G$1" x="97.79" y="91.44"/>
 <instance part="GND3" gate="1" x="22.86" y="76.2"/>
@@
 <instance part="GND6" gate="1" x="0" y="7.62"/>
 <instance part="R1" gate="G$1" x="73.66" y="50.8" rot="R270"/>
-<instance part="R3" gate="G$1" x="83.82" y="50.8" rot="R270"/>
+<instance part="R2" gate="G$1" x="83.82" y="50.8" rot="R270"/>
 <instance part="TXLED" gate="G$1" x="73.66" y="35.56"/>
 <instance part="RXLED" gate="G$1" x="83.82" y="35.56"/>
@@
 <instance part="C2" gate="G$1" x="48.26" y="91.44"/>
 <instance part="JP2" gate="G$1" x="66.04" y="0" rot="R180"/>
-<instance part="JP5" gate="G$1" x="45.72" y="2.54" rot="R180"/>
+<instance part="JP3" gate="G$1" x="45.72" y="2.54" rot="R180"/>
 </instances>
 <busses>
@@
 <pinref part="GND5" gate="1" pin="GND"/>
 <wire x1="115.57" y1="44.45" x2="115.57" y2="55.88" width="0.1524" layer="91"/>
-<pinref part="LED-P1.0" gate="G$1" pin="C"/>
+<pinref part="LED-P1.1" gate="G$1" pin="C"/>
 </segment>
 <segment>
@@
 </segment>
 <segment>
-<pinref part="C1" gate="G$1" pin="2"/>
+<pinref part="C3" gate="G$1" pin="2"/>
 <pinref part="GND6" gate="1" pin="GND"/>
 <wire x1="0" y1="25.4" x2="0" y2="10.16" width="0.1524" layer="91"/>
 </segment>
 <segment>
-<pinref part="C3" gate="G$1" pin="2"/>
+<pinref part="C1" gate="G$1" pin="2"/>
 <pinref part="GND3" gate="1" pin="GND"/>
 <wire x1="22.86" y1="88.9" x2="22.86" y2="86.36" width="0.1524" layer="91"/>
-<pinref part="JP3" gate="G$1" pin="GND"/>
 <wire x1="22.86" y1="86.36" x2="22.86" y2="78.74" width="0.1524" layer="91"/>
-<wire x1="5.08" y1="106.68" x2="15.24" y2="106.68" width="0.1524" layer="91"/>
-<wire x1="15.24" y1="106.68" x2="15.24" y2="86.36" width="0.1524" layer="91"/>
+<wire x1="15.24" y1="101.6" x2="15.24" y2="86.36" width="0.1524" layer="91"/>
 <wire x1="15.24" y1="86.36" x2="22.86" y2="86.36" width="0.1524" layer="91"/>
 <junction x="22.86" y="86.36"/>
@@
 <wire x1="48.26" y1="88.9" x2="48.26" y2="86.36" width="0.1524" layer="91"/>
 <wire x1="48.26" y1="86.36" x2="22.86" y2="86.36" width="0.1524" layer="91"/>
+<pinref part="JP1" gate="G$1" pin="VBUS"/>
+<wire x1="2.54" y1="101.6" x2="15.24" y2="101.6" width="0.1524" layer="91"/>
 </segment>
 <segment>
@@
 </segment>
 <segment>
-<pinref part="JP5" gate="G$1" pin="1"/>
+<pinref part="JP3" gate="G$1" pin="1"/>
 <wire x1="40.64" y1="5.08" x2="33.02" y2="5.08" width="0.1524" layer="91"/>
 </segment>
@@
 </segment>
 <segment>
-<pinref part="R2" gate="G$1" pin="2"/>
+<pinref part="R4" gate="G$1" pin="2"/>
 <pinref part="SUPPLY4" gate="1" pin="VCC"/>
 <wire x1="224.79" y1="88.9" x2="224.79" y2="82.55" width="0.1524" layer="91"/>
@@
 <pinref part="U2" gate="G$1" pin="3V3OUT"/>
 <wire x1="25.4" y1="43.18" x2="12.7" y2="43.18" width="0.1524" layer="91"/>
-<pinref part="C1" gate="G$1" pin="1"/>
+<pinref part="C3" gate="G$1" pin="1"/>
 <wire x1="12.7" y1="43.18" x2="0" y2="43.18" width="0.1524" layer="91"/>
 <wire x1="0" y1="43.18" x2="0" y2="33.02" width="0.1524" layer="91"/>
@@
 </segment>
 <segment>
-<pinref part="JP5" gate="G$1" pin="4"/>
+<pinref part="JP3" gate="G$1" pin="4"/>
 <wire x1="40.64" y1="-2.54" x2="33.02" y2="-2.54" width="0.1524" layer="91"/>
 </segment>
@@
 <net name="RESET" class="0">
 <segment>
-<pinref part="R2" gate="G$1" pin="1"/>
+<pinref part="R4" gate="G$1" pin="1"/>
 <wire x1="224.79" y1="72.39" x2="200.66" y2="72.39" width="0.1524" layer="91"/>
 <pinref part="U$1" gate="G$1" pin="24"/>
@@
 <segment>
 <wire x1="115.57" y1="68.58" x2="115.57" y2="63.5" width="0.1524" layer="91"/>
-<pinref part="LED-P1.0" gate="G$1" pin="A"/>
-<pinref part="R4" gate="G$1" pin="2"/>
+<pinref part="LED-P1.1" gate="G$1" pin="A"/>
+<pinref part="R3" gate="G$1" pin="2"/>
 </segment>
 </net>
@@
 </segment>
 <segment>
-<pinref part="JP5" gate="G$1" pin="2"/>
+<pinref part="JP3" gate="G$1" pin="2"/>
 <wire x1="40.64" y1="2.54" x2="33.02" y2="2.54" width="0.1524" layer="91"/>
 </segment>
@@
 </segment>
 <segment>
-<pinref part="JP5" gate="G$1" pin="3"/>
+<pinref part="JP3" gate="G$1" pin="3"/>
 <wire x1="40.64" y1="0" x2="33.02" y2="0" width="0.1524" layer="91"/>
 </segment>
@@
 <net name="N$13" class="0">
 <segment>
-<pinref part="R3" gate="G$1" pin="2"/>
+<pinref part="R2" gate="G$1" pin="2"/>
 <pinref part="RXLED" gate="G$1" pin="A"/>
 <wire x1="83.82" y1="45.72" x2="83.82" y2="38.1" width="0.1524" layer="91"/>
@@
 <net name="N$16" class="0">
 <segment>
-<pinref part="JP3" gate="G$1" pin="VBUS"/>
 <pinref part="L1" gate="G$1" pin="1"/>
 <wire x1="22.86" y1="104.14" x2="27.94" y2="104.14" width="0.1524" layer="91"/>
-<pinref part="C3" gate="G$1" pin="1"/>
+<pinref part="C1" gate="G$1" pin="1"/>
 <wire x1="22.86" y1="96.52" x2="22.86" y2="104.14" width="0.1524" layer="91"/>
+<pinref part="JP1" gate="G$1" pin="GND"/>
+<wire x1="2.54" y1="104.14" x2="22.86" y2="104.14" width="0.1524" layer="91"/>
 <junction x="22.86" y="104.14"/>
-<wire x1="22.86" y1="104.14" x2="5.08" y2="104.14" width="0.1524" layer="91"/>
 </segment>
 </net>
 <net name="USBDP" class="0">
 <segment>
-<pinref part="JP3" gate="G$1" pin="D-"/>
-<wire x1="5.08" y1="101.6" x2="12.7" y2="101.6" width="0.1524" layer="91"/>
+<pinref part="JP1" gate="G$1" pin="D-"/>
+<wire x1="2.54" y1="99.06" x2="7.62" y2="99.06" width="0.1524" layer="91"/>
 </segment>
 <segment>
@@
 <net name="USBDM" class="0">
 <segment>
-<pinref part="JP3" gate="G$1" pin="D+"/>
-<wire x1="5.08" y1="99.06" x2="12.7" y2="99.06" width="0.1524" layer="91"/>
+<pinref part="JP1" gate="G$1" pin="D+"/>
+<wire x1="2.54" y1="96.52" x2="7.62" y2="96.52" width="0.1524" layer="91"/>
 </segment>
 <segment>
@@
 <segment>
 <pinref part="U$1" gate="G$1" pin="2"/>
-<pinref part="R4" gate="G$1" pin="1"/>
+<pinref part="R3" gate="G$1" pin="1"/>
 <wire x1="153.67" y1="80.01" x2="115.57" y2="80.01" width="0.1524" layer="91"/>
 <wire x1="115.57" y1="80.01" x2="115.57" y2="78.74" width="0.1524" layer="91"/>
@@
 <pinref part="C2" gate="G$1" pin="1"/>
 <junction x="48.26" y="104.14"/>
-<pinref part="R3" gate="G$1" pin="1"/>
+<pinref part="R2" gate="G$1" pin="1"/>
 <wire x1="83.82" y1="66.04" x2="83.82" y2="55.88" width="0.1524" layer="91"/>
 <wire x1="48.26" y1="104.14" x2="83.82" y2="104.14" width="0.1524" layer="91"/>
