File: my-prj/MSP430_NRF24L01/V1_SENSOR.sch (EAGLE design)
At the start: 20 parts, among them U2 NRF24L01-4X2

Commit message: adding new files
Parts:
- removed R5: (no value), SparkFun-Passives:RESISTOR0805-RES
- removed R7: 220, SparkFun-Resistors:RESISTOR0805-RES
- removed U$3: MSP430G2553, TI_MSP430_v16:G2XX3---PW28
- added R103, R104: 47K, SparkFun-Resistors:RESISTOR0805-RES
- added U$1: TLV61220, custom:TI-TLV61220
- JP1: value M05X2PTH -> (none); device SparkFun-Connectors:M05X2PTH -> SparkFun-Connectors:M06LOCK
- JP2: value (none) -> M05X2PTH; device SparkFun-Connectors:M06LOCK -> SparkFun-Connectors:M05X2PTH
- R2: value 47K -> (none); device SparkFun-Resistors:RESISTOR0805-RES -> SparkFun-Passives:RESISTOR0805-RES
- R3: value 47K -> 220
- U$2: value TLV61220 -> MSP430G2553; device custom:TI-TLV61220 -> TI_MSP430_v16:G2XX3---PW28
- renumbered JP5 to JP3, LED-P3.0 to LED-P3.1, R10 to R101, R6 to R1, R8 to R102, R9 to R100, U2 to U1
Connections:
- net GND: now also JP1.6, JP2.1, JP2.3, JP2.5, JP2.7, JP2.9, R2.1, U$1.GND, U$2.28; no longer JP1.1, JP1.3, JP1.5, JP1.7, JP1.9, JP2.6, R5.1, U$2.GND, U$3.28
- net N$1: now also R103.1, R104.1, U$2.8; no longer R3.1, R4.1, U$3.8
- net N$13: now also U$1.SW; no longer U$2.SW
- net N$14: now also R2.2, U$1.FB; no longer R5.2, U$2.FB
- net N$15: now also R3.2; no longer R7.2
- net N$17: now also U$2.18; no longer U$3.18
- net N$18: now also U$2.17; no longer U$3.17
- net N$19: now also U$2.16; no longer U$3.16
- net N$20: now also U$2.11; no longer U$3.11
- net N$21: now also U$2.12; no longer U$3.12
- net N$22: now also U$2.10; no longer U$3.10
- net N$23: now also R3.1, U$2.9; no longer R7.1, U$3.9
- net P1.0: now also JP2.8, R103.2, U$2.2; no longer JP1.8, R4.2, U$3.2
- net P1.3: now also JP2.6, U$2.5; no longer JP1.6, U$3.5
- net P1.4: now also JP2.4, U$2.6; no longer JP1.4, U$3.6
- net P1.5: now also JP2.2, U$2.7; no longer JP1.2, U$3.7
- net P1.6: now also JP2.10, R104.2, U$2.22; no longer JP1.10, R3.2, U$3.22
- net RESET: now also JP1.5, R4.1, U$2.24; no longer JP2.5, R2.1, U$3.24
- net RXD: now also JP1.2, U$2.3; no longer JP2.2, U$3.3
- net TEST: now also JP1.4, U$2.25; no longer JP2.4, U$3.25
- net TXD: now also JP1.3, U$2.4; no longer JP2.3, U$3.4
- net VCC: now also C1.1, JP1.1, R4.2, U$1.VOUT, U$2.1; no longer C2.1, JP2.1, R2.2, U$2.VOUT, U$3.1
- net VIN: now also C2.1, U$1.EN, U$1.VBAT; no longer C1.1, U$2.EN, U$2.VBAT
Other:
- moved on the sheet: C1, C2, R2, R3, R4
